Commit message: Adding Last Updated Source File in Navigation

File: my_robot_ws/src/mybot_description/urdf/mybot2.xacro (robot description, xacro)
@@ -9,5 +9,5 @@
       <origin xyz="0 0 0" rpy=" 0 0 0"/>
       <geometry>
-        <box size=".6 .3 .1"/>
+        <box size=".6 .5 .136"/>
       </geometry>
     </visual>
@@ -23,11 +23,11 @@
    <collision name='collision'>
       <geometry>
-        <box size=".6 .3 .1"/>
+        <box size=".6 .5 .136"/>
       </geometry>
    </collision>
  <collision name='caster_collision'>
-    <origin xyz="-0.2 0 -0.05" rpy=" 0 0 0"/>
+    <origin xyz="-0.25 0 -0.068" rpy=" 0 0 0"/>
     <geometry>
-        <sphere radius="0.05"/>
+        <sphere radius="0.0402"/>
     </geometry>
     <surface>
@@ -43,7 +43,29 @@
  </collision>
 <visual name='caster_visual'>
-     <origin xyz="-0.2 0 -0.05" rpy=" 0 0 0"/>
+     <origin xyz="-0.25 0 -0.068" rpy=" 0 0 0"/>
      <geometry>
-      <sphere radius="0.05"/>
+      <sphere radius="0.0402"/>
+     </geometry>
+</visual>
+ <collision name='caster2_collision'>
+    <origin xyz="0.25 0 -0.068" rpy=" 0 0 0"/>
+    <geometry>
+        <sphere radius="0.0402"/>
+    </geometry>
+    <surface>
+        <friction>
+          <ode>
+            <mu>0</mu>
+            <mu2>0</mu2>
+            <slip1>1.0</slip1>
+            <slip2>1.0</slip2>
+          </ode>
+        </friction>
+     </surface>
+ </collision>
+<visual name='caster2_visual'>
+     <origin xyz="0.25 0 -0.068" rpy=" 0 0 0"/>
+     <geometry>
+      <sphere radius="0.0402"/>
      </geometry>
 </visual>
@@ -52,5 +74,5 @@
 <!--left wheel Joint /-->
   <joint type="continuous" name="left_wheel_hinge">
-    <origin xyz="0.1 0.175 0" rpy="0 0 0"/>
+    <origin xyz="0 0.1895 -0.0317" rpy="0 0 0"/>
     <child link="left_wheel"/>
     <parent link="chassis"/>
@@ -64,5 +86,5 @@
       <origin xyz="0 0 0" rpy="0 1.5707 1.5707"/>
       <geometry>
-        <cylinder radius="0.1" length="0.05"/>
+        <cylinder radius="0.0765" length="0.035"/>
       </geometry>
     </visual>
@@ -70,5 +92,5 @@
       <origin xyz="0 0 0" rpy="0 1.5707 1.5707"/>
       <geometry>
-        <cylinder radius="0.1" length="0.05"/>
+        <cylinder radius="0.0765" length="0.035"/>
       </geometry>
     </collision>
@@ -76,5 +98,5 @@
       <origin xyz="0 0 0" rpy="0 1.5707 1.5707"/>
       <mass value="5"/>
-      <cylinder_inertia m="5" r="0.1" h="0.05"/>
+      <cylinder_inertia m="5" r="0.0765" h="0.035"/>
       <inertia
         ixx="1.0" ixy="0.0" ixz="0.0"
@@ -86,5 +108,5 @@
 <!--Right wheel joint/-->
   <joint type="continuous" name="right_wheel_hinge">
-    <origin xyz="0.1 -0.175 0" rpy="0 0 0"/>
+    <origin xyz="0 -0.1895 -0.0317" rpy="0 0 0"/>
     <child link="right_wheel"/>
     <parent link="chassis"/>
@@ -98,5 +120,5 @@
       <origin xyz="0 0 0" rpy="0 1.5707 1.5707"/>
       <geometry>
-        <cylinder radius="0.1" length="0.05"/>
+        <cylinder radius="0.0765" length="0.035"/>
       </geometry>
     </visual>
@@ -104,5 +126,5 @@
       <origin xyz="0 0 0" rpy="0 1.5707 1.5707"/>
       <geometry>
-        <cylinder radius="0.1" length="0.05"/>
+        <cylinder radius="0.0765" length="0.035"/>
       </geometry>
     </collision>
@@ -110,5 +132,5 @@
       <origin xyz="0 0 0" rpy="0 1.5707 1.5707"/>
       <mass value="5"/>
-      <cylinder_inertia m="5" r="0.1" h="0.05"/>
+      <cylinder_inertia m="5" r="0.0765" h="0.035"/>
       <inertia
         ixx="1.0" ixy="0.0" ixz="0.0"
@@ -117,8 +139,38 @@
       </inertial>
   </link>
+  <!-- ++++++++++++++++++  Upper level  +++++++++++++++++++++++++++++ /-->
+<!--upper level joint /-->
+<joint name="upper_level_joint" type="fixed">
+    <origin xyz="0 0 0.206" rpy="0 0 0"/>
+    <parent link="chassis"/>
+    <child link="upper_level"/>
+</joint>
+<!--upper level  Link /-->
+<link name="upper_level">
+	<visual>
+            <geometry>
+        	<box size=".6 .5 .136"/>
+      	    </geometry>
+            <material name="red"/>
+        </visual>
+        <inertial>
+      <mass value="10.0"/>
+      <origin xyz="0 0 0" rpy=" 0 0 0"/>
+      <inertia
+          ixx="0.5" ixy="0" ixz="0"
+          iyy="1.0" iyz="0"
+          izz="0.1"
+      />
+   </inertial>
+   <collision name='collision'>
+      <geometry>
+        <box size=".6 .5 .136"/>
+      </geometry>
+   </collision>
+</link>
 <!-- ++++++++++++++++++  rplidar  +++++++++++++++++++++++++++++ /-->
 <!--rplidar joint /-->
 <joint name="rplidar_joint" type="fixed">
-    <origin xyz=".15 0 .1" rpy="0 0 0"/>
+    <origin xyz="0.065 0 0.098" rpy="0 0 0"/>
     <parent link="chassis"/>
     <child link="rplidar_link"/>
@@ -128,5 +180,5 @@
 	<visual>
             <geometry>
-                <cylinder radius="0.05" length="0.07"/>
+                <cylinder radius="0.05" length="0.06"/>
             </geometry>
             <material name="red"/>
@@ -134,71 +186,98 @@
         <collision>
             <geometry>
-                <cylinder radius="0.05" length="0.07"/>
-            </geometry>
-        </collision>
-        <xacro:inertial_cylinder mass="0.1" length="0.07" radius="0.05">
-            <origin xyz="0 0 0" rpy="0 0 0"/>
-        </xacro:inertial_cylinder>
-</link>
-	<!--  ++++++++++++++++++Gazebo Plugins+++++++++++++++++++          /-->
-<gazebo>
-    <plugin name="differential_drive_controller" filename="libgazebo_ros_diff_drive.so">
-      <legacyMode>false</legacyMode>
-      <alwaysOn>true</alwaysOn>
-      <updateRate>20</updateRate>
-      <leftJoint>left_wheel_hinge</leftJoint>
-      <rightJoint>right_wheel_hinge</rightJoint>
-      <publishWheelJointState>true</publishWheelJointState>
-      <wheelSeparation>0.4</wheelSeparation>
-      <wheelDiameter>0.1</wheelDiameter>
-      <Torque>20</Torque>
-      <commandTopic>cmd_vel</commandTopic> <!--   listening to the topic "cmd_vel"   : to move the robot      /-->
-      <odometryTopic>odom</odometryTopic>
-      <odometryFrame>odom</odometryFrame>
-      <robotBaseFrame>chassis</robotBaseFrame>
-    <!--  <publish_odom>true</publish_odom>
-      <publishOdomTF>true</publishOdomTF>
-      <publishWheelTF>true</publishWheelTF>
-/-->
-      </plugin>
- </gazebo>
-<!--  +++++++++++++Chassis Orange color++++++++++++++++          /-->
-  <gazebo reference="chassis">
-    <material>Gazebo/Orange</material>
-  </gazebo>
-<!--  ++++++++++++++++Left wheel Blue Color+++++++++++++++++++          /-->
-  <gazebo reference="left_wheel">
-    <material>Gazebo/Blue</material>
-  </gazebo>
-<!--  +++++++++++++++Right wheel Blue Color+++++++++++++++++          /-->
-  <gazebo reference="right_wheel">
-    <material>Gazebo/Blue</material>
-  </gazebo>
-<!--  ++++++++++++++++++rplidar Plugin+++++++++++++++++++          /-->
-<gazebo reference="rplidar_link">
-	<material>Gazebo/Red</material>
-        <sensor name="laser" type="ray">
-            <pose> 0 0 0 0 0 0 </pose>
-            <visualize>true</visualize>
-            <update_rate>5.5</update_rate>
-            <ray>
-                <scan>
-                    <horizontal>
-                        <samples>2048</samples>
-                        <min_angle>-3.14</min_angle>
-                        <max_angle>3.14</max_angle>
-                    </horizontal>
-                </scan>
-                <range>
-                    <min>0.3</min>
-                    <max>12</max>
-                </range>
-            </ray>
-            <plugin name="laser_controller" filename="libgazebo_ros_laser.so">
-                <output_type>sensor_msgs/LaserScan</output_type>
-                <topicName>/scan</topicName>
-                <frameName>rplidar_link</frameName>
-            </plugin>
-        </sensor>
-</gazebo>
+                <cylinder radius="0.05" length="0.06"/>
+            </geometry>
+        </collision>
+        <xacro:inertial_cylinder mass="0.1" length="0.06" radius="0.05">
+            <origin xyz="0 0 0" rpy="0 0 0"/>
+        </xacro:inertial_cylinder>
+</link>
+<!-- ++++++++++++++++++Four Supports++++++++++++++++++++ /-->
+<joint name="support1_joint" type="fixed">
+    <origin xyz="0.28 0.22 0.103" rpy="0 0 0"/>
+    <parent link="chassis"/>
+    <child link="support1_link"/>
+</joint>
+<link name="support1_link">
+	<visual>
+            <geometry>
+                <cylinder radius="0.008" length="0.07"/>
+            </geometry>
+            <material name="green"/>
+        </visual>
+        <collision>
+            <geometry>
+                <cylinder radius="0.008" length="0.07"/>
+            </geometry>
+        </collision>
+        <xacro:inertial_cylinder mass="0.1" length="0.07" radius="0.008">
+            <origin xyz="0 0 0" rpy="0 0 0"/>
+        </xacro:inertial_cylinder>
+</link>
+<!--++++++++++++++++++++++++++++++++++++++++++++++++++++++ /-->
+<joint name="support2_joint" type="fixed">
+    <origin xyz="-0.28 0.22 0.103" rpy="0 0 0"/>
+    <parent link="chassis"/>
+    <child link="support2_link"/>
+</joint>
+<link name="support2_link">
+	<visual>
+            <geometry>
+                <cylinder radius="0.008" length="0.07"/>
+            </geometry>
+            <material name="green"/>
+        </visual>
+        <collision>
+            <geometry>
+                <cylinder radius="0.008" length="0.07"/>
+            </geometry>
+        </collision>
+        <xacro:inertial_cylinder mass="0.1" length="0.07" radius="0.008">
+            <origin xyz="0 0 0" rpy="0 0 0"/>
+        </xacro:inertial_cylinder>
+</link>
+<!--++++++++++++++++++++++++++++++++++++++++++++++++++++++ /-->
+<joint name="support3_joint" type="fixed">
+    <origin xyz="-0.28 -0.22 0.103" rpy="0 0 0"/>
+    <parent link="chassis"/>
+    <child link="support3_link"/>
+</joint>
+<link name="support3_link">
+	<visual>
+            <geometry>
+                <cylinder radius="0.008" length="0.07"/>
+            </geometry>
+            <material name="green"/>
+        </visual>
+        <collision>
+            <geometry>
+                <cylinder radius="0.008" length="0.07"/>
+            </geometry>
+        </collision>
+        <xacro:inertial_cylinder mass="0.1" length="0.07" radius="0.008">
+            <origin xyz="0 0 0" rpy="0 0 0"/>
+        </xacro:inertial_cylinder>
+</link>
+<!--++++++++++++++++++++++++++++++++++++++++++++++++++++++ /-->
+<joint name="support4_joint" type="fixed">
+    <origin xyz="0.28 -0.22 0.103" rpy="0 0 0"/>
+    <parent link="chassis"/>
+    <child link="support4_link"/>
+</joint>
+<link name="support4_link">
+	<visual>
+            <geometry>
+                <cylinder radius="0.008" length="0.07"/>
+            </geometry>
+            <material name="green"/>
+        </visual>
+        <collision>
+            <geometry>
+                <cylinder radius="0.008" length="0.07"/>
+            </geometry>
+        </collision>
+        <xacro:inertial_cylinder mass="0.1" length="0.07" radius="0.008">
+            <origin xyz="0 0 0" rpy="0 0 0"/>
+        </xacro:inertial_cylinder>
+</link>
 </robot>
